Commit message: arrange

File: pr2hand/pr2hand.urdf (robot description, URDF)
Before this commit: robot pr2hand, 10 links, 9 joints
Links:
- added link r_gripper_l_finger_tip_frame
- added link r_gripper_l_keypoint1_link
- added link r_gripper_r_keypoint1_link
Joints:
- added joint r_gripper_joint: type prismatic, parent r_gripper_r_finger_tip_link, child r_gripper_l_finger_tip_frame, axis 0 1 0, limit lower=0.0 upper=0.09 effort=1000.0 velocity=0.2
- added joint r_gripper_l_keypoint1_joint: type revolute, parent r_gripper_l_finger_link, child r_gripper_l_keypoint1_link, origin xyz=0.071 0.0032 0.0 rpy=0 0 0, axis 0 0 1, limit lower=0.0 upper=0.548 effort=1000.0 velocity=0.5
- added joint r_gripper_r_keypoint1_joint: type revolute, parent r_gripper_r_finger_link, child r_gripper_r_keypoint1_link, origin xyz=0.071 -0.0032 0.0 rpy=0 0 0, axis 0 0 1, limit lower=0.0 upper=0.548 effort=1000.0 velocity=0.5

File: pr2hand/pr2hand_for_check.urdf (robot description, URDF)
Before this commit: robot pr2hand, 11 links, 10 joints
Links:
- added link r_gripper_l_keypoint1_link
- added link r_gripper_r_keypoint1_link
Joints:
- added joint r_gripper_l_keypoint1_joint: type revolute, parent r_gripper_l_finger_link, child r_gripper_l_keypoint1_link, origin xyz=0.071 0.0032 0.0 rpy=0 0 0, axis 0 0 1, limit lower=0.0 upper=0.548 effort=1000.0 velocity=0.5
- added joint r_gripper_r_keypoint1_joint: type revolute, parent r_gripper_r_finger_link, child r_gripper_r_keypoint1_link, origin xyz=0.071 -0.0032 0.0 rpy=0 0 0, axis 0 0 1, limit lower=0.0 upper=0.548 effort=1000.0 velocity=0.5

File: pr2hand/robots/pr2hand.urdf.xacro (robot description, xacro)
@@ -8,10 +8,8 @@
   <xacro:include filename="$(find pr2_description)/urdf/sensors/projector_wg6802418.urdf.xacro" />
   <!-- generic simulator_gazebo plugins for starting mechanism control, ros time, ros battery -->
-  <xacro:include filename="$(find pr2_description)/gazebo/gazebo.urdf.xacro" />
+  <!-- <xacro:include filename="$(find pr2_description)/gazebo/gazebo.urdf.xacro" /> -->
   <!-- materials for visualization -->
   <xacro:include filename="$(find pr2_description)/urdf/materials.urdf.xacro" />
-  <xacro:include filename="$(find pr2_description)/urdf/base_v0/base.urdf.xacro" />
   <!-- use gripper as base  -->
-  <!-- <xacro:pr2_base_v0 name="base"/> -->
   <xacro:pr2_gripper_v0 reflect="-1.0" side="r" name="base"
                screw_reduction="${4.0/1000.0}"

Commit message: add kp2

File: pr2hand/pr2hand.urdf (robot description, URDF)
Before this commit: robot pr2hand, 13 links, 12 joints
Links:
- added link r_gripper_l_keypoint2_link
- added link r_gripper_r_keypoint2_link
Joints:
- added joint r_gripper_l_keypoint2_joint: type fixed, parent base_link, child r_gripper_l_keypoint2_link, origin xyz=0.119 0.007 0.0 rpy=0 0 0, axis 0 0 1
- added joint r_gripper_r_keypoint2_joint: type fixed, parent base_link, child r_gripper_r_keypoint2_link, origin xyz=0.119 -0.007 0.0 rpy=0 0 0, axis 0 0 1

File: pr2hand/pr2hand_for_check.urdf (robot description, URDF)
Before this commit: robot pr2hand, 13 links, 12 joints
Links:
- added link r_gripper_l_keypoint2_link
- added link r_gripper_r_keypoint2_link
Joints:
- added joint r_gripper_l_keypoint2_joint: type fixed, parent base_link, child r_gripper_l_keypoint2_link, origin xyz=0.119 0.007 0.0 rpy=0 0 0, axis 0 0 1
- added joint r_gripper_r_keypoint2_joint: type fixed, parent base_link, child r_gripper_r_keypoint2_link, origin xyz=0.119 -0.007 0.0 rpy=0 0 0, axis 0 0 1
